Commit message: Rectified rpy values for origins of arms in gripper.

File: urdf/gripper.xacro (robot description, xacro)
@@ -56,5 +56,5 @@
       </inertial>
       <visual>
-        <origin  xyz="0 0 0" rpy="0 0 0" />
+        <origin  xyz="0 0 0" rpy="0.7854 0 3.1416" />
         <geometry>
             <mesh filename="package://swarm_collection/meshes/arm_link.STL" scale="1 1 1" />
@@ -90,5 +90,5 @@
       </inertial>
       <visual>
-        <origin  xyz="0 0 0" rpy="0 0 0" />
+        <origin  xyz="0 0 0" rpy="0.7854 0 -1.0472" />
         <geometry>
             <mesh filename="package://swarm_collection/meshes/arm_link.STL" scale="1 1 1" />
@@ -124,5 +124,5 @@
       </inertial>
       <visual>
-        <origin  xyz="0 0 0" rpy="0 0 0" />
+        <origin  xyz="0 0 0" rpy="0.7854 0 1.0472" />
         <geometry>
             <mesh filename="package://swarm_collection/meshes/arm_link.STL" scale="1 1 1" />

Commit message: Stabilized the Drone at Startup of Program Exectution

File: urdf/gripper.xacro (robot description, xacro)
@@ -1,4 +1,21 @@
 <?xml version="1.0"?>
 <robot xmlns:xacro="http://ros.org/wiki/xacro">
+<!-- mass of arm = 0.12781 -->
+<!-- Inertia of Hub
+<inertia
+  ixx="2.575E-05"
+  ixy="-6.389E-10"
+  ixz="2.3003E-11"
+  iyy="2.5749E-05"
+  iyz="3.7001E-10"
+  izz="4.5243E-05" /> -->
+  <!-- Inertia of Arm
+ <inertia
+    ixx="0.00027224"
+    ixy="-6.26E-11"
+    ixz="-5.2198E-10"
+    iyy="0.00022223"
+    iyz="-7.6551E-05"
+    izz="6.3032E-05" /> -->
 <!--for hub -->
   <xacro:macro name="hub_macro"
@@ -14,10 +31,10 @@
         <mass value="0.031918" /> <!-- [kg] -->
         <inertia
-          ixx="2.575E-05"
-          ixy="-6.389E-10"
-          ixz="2.3003E-11"
-          iyy="2.5749E-05"
-          iyz="3.7001E-10"
-          izz="4.5243E-05" />
+          ixx="255.496140E-6"
+          ixy="-0.048915E-6"
+          ixz="-0.024520E-6"
+          iyy="255.632690E-6"
+          iyz="0.105558E-6"
+          izz="448.948303E-6" />
       </inertial>
       <visual>
@@ -28,4 +45,5 @@
       </visual>
       <collision>
+        <origin  xyz="0 0 0" rpy="0 0 0" />
         <geometry>
           <mesh
@@ -46,12 +64,12 @@
     <link name="${robot_namespace}/ARM1">
       <inertial>
-        <mass value="0.12781" /> <!-- [kg] -->
+        <mass value="0.05" /> <!-- [kg] -->
         <inertia
-          ixx="0.00027224"
-          ixy="-6.26E-11"
-          ixz="-5.2198E-10"
-          iyy="0.00022223"
-          iyz="-7.6551E-05"
-          izz="6.3032E-05" />
+          ixx="2714.030518E-6"
+          ixy="0.000007E-6"
+          ixz="0.000038E-6"
+          iyy="2216.979248E-6"
+          iyz="-762.669067E-6"
+          izz="627.139465E-6" />
       </inertial>
       <visual>
@@ -62,4 +80,5 @@
       </visual>
       <collision>
+        <origin  xyz="0 0 0" rpy="0.7854 0 3.1416" />
         <geometry>
           <mesh
@@ -80,12 +99,12 @@
     <link name="${robot_namespace}/ARM2">
       <inertial>
-        <mass value="0.12781" /> <!-- [kg] -->
+        <mass value="0.05" /> <!-- [kg] -->
         <inertia
-          ixx="0.00027224"
-          ixy="-6.26E-11"
-          ixz="-5.2198E-10"
-          iyy="0.00022223"
-          iyz="-7.6551E-05"
-          izz="6.3032E-05" />
+          ixx="2714.030518E-6"
+          ixy="0.000007E-6"
+          ixz="0.000038E-6"
+          iyy="2216.979248E-6"
+          iyz="-762.669067E-6"
+          izz="627.139465E-6" />
       </inertial>
       <visual>
@@ -96,4 +115,5 @@
       </visual>
       <collision>
+        <origin  xyz="0 0 0" rpy="0.7854 0 -1.0472" />
         <geometry>
           <mesh
@@ -114,12 +134,12 @@
     <link name="${robot_namespace}/ARM3">
       <inertial>
-        <mass value="0.12781" /> <!-- [kg] -->
+        <mass value="0.05" /> <!-- [kg] -->
         <inertia
-          ixx="0.00027224"
-          ixy="-6.26E-11"
-          ixz="-5.2198E-10"
-          iyy="0.00022223"
-          iyz="-7.6551E-05"
-          izz="6.3032E-05" />
+          ixx="2714.030518E-6"
+          ixy="0.000007E-6"
+          ixz="0.000038E-6"
+          iyy="2216.979248E-6"
+          iyz="-762.669067E-6"
+          izz="627.139465E-6" />
       </inertial>
       <visual>
@@ -130,4 +150,5 @@
       </visual>
       <collision>
+        <origin  xyz="0 0 0" rpy="0.7854 0 1.0472" />
         <geometry>
           <mesh

File: urdf/iris.xacro (robot description, xacro)
@@ -1,33 +1,20 @@
 <?xml version="1.0"?>
-<!--
-  Copyright 2015 Fadri Furrer, ASL, ETH Zurich, Switzerland
-  Copyright 2015 Michael Burri, ASL, ETH Zurich, Switzerland
-  Copyright 2015 Mina Kamel, ASL, ETH Zurich, Switzerland
-  Copyright 2015 Janosch Nikolic, ASL, ETH Zurich, Switzerland
-  Copyright 2015 Markus Achtelik, ASL, ETH Zurich, Switzerland
-  Licensed under the Apache License, Version 2.0 (the "License");
-  you may not use this file except in compliance with the License.
-  You may obtain a copy of the License at
-  http://www.apache.org/licenses/LICENSE-2.0
-  Unless required by applicable law or agreed to in writing, software
-  distributed under the License is distributed on an "AS IS" BASIS,
-  WITHOUT WARRANTIES OR CONDITIONS OF ANY KIND, either express or implied.
-  See the License for the specific language governing permissions and
-  limitations under the License.
--->
-<robot name="firefly" xmlns:xacro="http://ros.org/wiki/xacro">
+<robot name="iris" xmlns:xacro="http://ros.org/wiki/xacro">
   <!-- Properties -->
   <xacro:property name="namespace" value="$(arg namespace)" />
   <xacro:property name="rotor_velocity_slowdown_sim" value="10" />
   <xacro:property name="use_mesh_file" value="true" />
-  <xacro:property name="mesh_file" value="package://swarm_collection/meshes/firefly.stl" />
+  <xacro:property name="mesh_file" value="package://rotors_description/meshes/iris.dae" />
   <xacro:property name="mass" value="1.5" /> <!-- [kg] -->
-  <xacro:property name="body_width" value="0.1" /> <!-- [m] -->
-  <xacro:property name="body_height" value="0.16" /> <!-- [m] -->
+  <xacro:property name="body_width" value="0.47" /> <!-- [m] -->
+  <xacro:property name="body_height" value="0.11" /> <!-- [m] -->
   <xacro:property name="mass_rotor" value="0.005" /> <!-- [kg] -->
-  <xacro:property name="arm_length" value="0.215" /> <!-- [m] -->
-  <xacro:property name="rotor_offset_top" value="0.037" /> <!-- [m] -->
+  <xacro:property name="arm_length_front_x" value="0.13" /> <!-- [m] -->
+  <xacro:property name="arm_length_back_x" value="0.13" /> <!-- [m] -->
+  <xacro:property name="arm_length_front_y" value="0.22" /> <!-- [m] -->
+  <xacro:property name="arm_length_back_y" value="0.2" /> <!-- [m] -->
+  <xacro:property name="rotor_offset_top" value="0.023" /> <!-- [m] -->
   <xacro:property name="radius_rotor" value="0.1" /> <!-- [m] -->
-  <xacro:property name="motor_constant" value="8.54858e-06" /> <!-- [kg m/s^2] -->
+  <xacro:property name="motor_constant" value="8.54858e-06" /> <!-- [kg.m/s^2] -->
   <xacro:property name="moment_constant" value="0.016" /> <!-- [m] -->
   <xacro:property name="time_constant_up" value="0.0125" /> <!-- [s] -->
@@ -36,9 +23,10 @@
   <xacro:property name="sin30" value="0.5" />
   <xacro:property name="cos30" value="0.866025403784" />
+  <xacro:property name="sqrt2" value="1.4142135623730951" />
   <xacro:property name="rotor_drag_coefficient" value="8.06428e-05" />
   <xacro:property name="rolling_moment_coefficient" value="0.000001" />
   <!-- Property Blocks -->
   <xacro:property name="body_inertia">
-    <inertia ixx="0.0347563" ixy="0.0" ixz="0.0" iyy="0.0458929" iyz="0.0" izz="0.0977" /> <!-- [kg m^2] [kg m^2] [kg m^2] [kg m^2] [kg m^2] [kg m^2] -->
+    <inertia ixx="0.0347563" ixy="0.0" ixz="0.0" iyy="0.0458929" iyz="0.0" izz="0.0977" /> <!-- [kg.m^2] [kg.m^2] [kg.m^2] [kg.m^2] [kg.m^2] [kg.m^2] -->
   </xacro:property>
   <!-- inertia of a single rotor, assuming it is a cuboid. Height=3mm, width=15mm -->
@@ -63,5 +51,5 @@
   <xacro:vertical_rotor
     robot_namespace="${namespace}"
-    suffix="front_left"
+    suffix="front_right"
     direction="ccw"
     motor_constant="${motor_constant}"
@@ -76,32 +64,12 @@
     rotor_drag_coefficient="${rotor_drag_coefficient}"
     rolling_moment_coefficient="${rolling_moment_coefficient}"
-    color="Red"
-    use_own_mesh="false"
-    mesh="">
-    <origin xyz="${cos30*arm_length} ${sin30*arm_length} ${rotor_offset_top}" rpy="0 0 0" />
+    color="Blue"
+    use_own_mesh="false"
+    mesh="">
+    <origin xyz="${arm_length_front_x} -${arm_length_front_y} ${rotor_offset_top}" rpy="0 0 0" />
     <xacro:insert_block name="rotor_inertia" />
   </xacro:vertical_rotor>
   <xacro:vertical_rotor
     robot_namespace="${namespace}"
-    suffix="left"
-    direction="cw"
-    motor_constant="${motor_constant}"
-    moment_constant="${moment_constant}"
-    parent="${namespace}/base_link"
-    mass_rotor="${mass_rotor}"
-    radius_rotor="${radius_rotor}"
-    time_constant_up="${time_constant_up}"
-    time_constant_down="${time_constant_down}"
-    max_rot_velocity="${max_rot_velocity}"
-    motor_number="1"
-    rotor_drag_coefficient="${rotor_drag_coefficient}"
-    rolling_moment_coefficient="${rolling_moment_coefficient}"
-    color="Blue"
-    use_own_mesh="false"
-    mesh="">
-    <origin xyz="0 ${arm_length} ${rotor_offset_top}" rpy="0 0 0" />
-    <xacro:insert_block name="rotor_inertia" />
-  </xacro:vertical_rotor>
-  <xacro:vertical_rotor robot_namespace="${namespace}"
     suffix="back_left"
     direction="ccw"
@@ -114,4 +82,24 @@
     time_constant_down="${time_constant_down}"
     max_rot_velocity="${max_rot_velocity}"
+    motor_number="1"
+    rotor_drag_coefficient="${rotor_drag_coefficient}"
+    rolling_moment_coefficient="${rolling_moment_coefficient}"
+    color="Red"
+    use_own_mesh="false"
+    mesh="">
+    <origin xyz="-${arm_length_back_x} ${arm_length_back_y} ${rotor_offset_top}" rpy="0 0 0" />
+    <xacro:insert_block name="rotor_inertia" />
+  </xacro:vertical_rotor>
+  <xacro:vertical_rotor robot_namespace="${namespace}"
+    suffix="front_left"
+    direction="cw"
+    motor_constant="${motor_constant}"
+    moment_constant="${moment_constant}"
+    parent="${namespace}/base_link"
+    mass_rotor="${mass_rotor}"
+    radius_rotor="${radius_rotor}"
+    time_constant_up="${time_constant_up}"
+    time_constant_down="${time_constant_down}"
+    max_rot_velocity="${max_rot_velocity}"
     motor_number="2"
     rotor_drag_coefficient="${rotor_drag_coefficient}"
@@ -120,5 +108,5 @@
     use_own_mesh="false"
     mesh="">
-    <origin xyz="-${cos30*arm_length} ${sin30*arm_length} ${rotor_offset_top}" rpy="0 0 0" />
+    <origin xyz="${arm_length_front_x} ${arm_length_front_y} ${rotor_offset_top}" rpy="0 0 0" />
     <xacro:insert_block name="rotor_inertia" />
   </xacro:vertical_rotor>
@@ -137,32 +125,37 @@
     rotor_drag_coefficient="${rotor_drag_coefficient}"
     rolling_moment_coefficient="${rolling_moment_coefficient}"
-    color="Blue"
-    use_own_mesh="false"
-    mesh="">
-    <origin xyz="-${cos30*arm_length} -${sin30*arm_length} ${rotor_offset_top}" rpy="0 0 0" />
-    <xacro:insert_block name="rotor_inertia" />
-  </xacro:vertical_rotor>
-  <xacro:vertical_rotor
-    robot_namespace="${namespace}"
-    suffix="right"
-    direction="ccw"
-    motor_constant="${motor_constant}"
-    moment_constant="${moment_constant}"
-    parent="${namespace}/base_link"
-    mass_rotor="${mass_rotor}"
-    radius_rotor="${radius_rotor}"
-    time_constant_up="${time_constant_up}"
-    time_constant_down="${time_constant_down}"
-    max_rot_velocity="${max_rot_velocity}"
-    motor_number="4"
-    rotor_drag_coefficient="${rotor_drag_coefficient}"
-    rolling_moment_coefficient="${rolling_moment_coefficient}"
-    color="Blue"
-    use_own_mesh="false"
-    mesh="">
-    <origin xyz="0 -${arm_length} ${rotor_offset_top}" rpy="0 0 0" />
-    <xacro:insert_block name="rotor_inertia" />
-  </xacro:vertical_rotor>
-  <xacro:vertical_rotor
+    color="Red"
+    use_own_mesh="false"
+    mesh="">
+    <origin xyz="-${arm_length_back_x} -${arm_length_back_y} ${rotor_offset_top}" rpy="0 0 0" />
+    <xacro:insert_block name="rotor_inertia" />
+  </xacro:vertical_rotor>
+  <!-- for hub -->
+    <xacro:hub_macro
+      robot_namespace="${namespace}"
+      suffix="front_right"
+      direction="cw"
+      motor_constant="${motor_constant}"
+      moment_constant="${moment_constant}"
+      parent="${namespace}/base_link"
+      mass_rotor="${mass_rotor}"
+      radius_rotor="${radius_rotor}"
+      time_constant_up="${time_constant_up}"
+      time_constant_down="${time_constant_down}"
+      max_rot_velocity="${max_rot_velocity}"
+      motor_number="5"
+      rotor_drag_coefficient="${rotor_drag_coefficient}"
+      rolling_moment_coefficient="${rolling_moment_coefficient}"
+      color="Red"
+      use_own_mesh="false"
+      mesh="">
+      <origin xyz="0 0 -0.02" rpy="0 0 0.5236" />
+      <xacro:insert_block name="rotor_inertia" />
+    </xacro:hub_macro>
+    <!-- Pi/3 = 1.0472 -->
+    <!-- Pi/2 = 1.5708 -->
+    <!-- Pi/6 = 0.5236 -->
+  <!-- for ARM1 -->
+  <xacro:ARM1_macro
     robot_namespace="${namespace}"
     suffix="front_right"
@@ -182,9 +175,9 @@
     use_own_mesh="false"
     mesh="">
-    <origin xyz="${cos30*arm_length} -${sin30*arm_length} ${rotor_offset_top}" rpy="0 0 0" />
-    <xacro:insert_block name="rotor_inertia" />
-  </xacro:vertical_rotor>
-<!-- for hub -->
-  <xacro:hub_macro
+    <origin xyz="0 -0.0225 -0.03" rpy="0 0 0" />
+    <xacro:insert_block name="rotor_inertia" />
+  </xacro:ARM1_macro>
+  <!-- for ARM2 -->
+  <xacro:ARM2_macro
     robot_namespace="${namespace}"
     suffix="front_right"
@@ -204,75 +197,28 @@
     use_own_mesh="false"
     mesh="">
-    <origin xyz="0 0 0" rpy="0 0 0.5236" />
-    <xacro:insert_block name="rotor_inertia" />
-  </xacro:hub_macro>
-  <!-- Pi/3 = 1.0472 -->
-  <!-- Pi/2 = 1.5708 -->
-  <!-- Pi/6 = 0.5236 -->
-<!-- for ARM1 -->
-<xacro:ARM1_macro
-  robot_namespace="${namespace}"
-  suffix="front_right"
-  direction="cw"
-  motor_constant="${motor_constant}"
-  moment_constant="${moment_constant}"
-  parent="${namespace}/base_link"
-  mass_rotor="${mass_rotor}"
-  radius_rotor="${radius_rotor}"
-  time_constant_up="${time_constant_up}"
-  time_constant_down="${time_constant_down}"
-  max_rot_velocity="${max_rot_velocity}"
-  motor_number="5"
-  rotor_drag_coefficient="${rotor_drag_coefficient}"
-  rolling_moment_coefficient="${rolling_moment_coefficient}"
-  color="Red"
-  use_own_mesh="false"
-  mesh="">
-  <origin xyz="0 -0.0225 -0.03" rpy="0 0 0" />
-  <xacro:insert_block name="rotor_inertia" />
-</xacro:ARM1_macro>
-<!-- for ARM2 -->
-<xacro:ARM2_macro
-  robot_namespace="${namespace}"
-  suffix="front_right"
-  direction="cw"
-  motor_constant="${motor_constant}"
-  moment_constant="${moment_constant}"
-  parent="${namespace}/base_link"
-  mass_rotor="${mass_rotor}"
-  radius_rotor="${radius_rotor}"
-  time_constant_up="${time_constant_up}"
-  time_constant_down="${time_constant_down}"
-  max_rot_velocity="${max_rot_velocity}"
-  motor_number="5"
-  rotor_drag_coefficient="${rotor_drag_coefficient}"
-  rolling_moment_coefficient="${rolling_moment_coefficient}"
-  color="Red"
-  use_own_mesh="false"
-  mesh="">
-  <origin xyz="0.01948557158 0.01125 -0.03" rpy="0 0 0" />
-  <xacro:insert_block name="rotor_inertia" />
-</xacro:ARM2_macro>
-<!-- for ARM3 -->
-<xacro:ARM3_macro
-  robot_namespace="${namespace}"
-  suffix="front_right"
-  direction="cw"
-  motor_constant="${motor_constant}"
-  moment_constant="${moment_constant}"
-  parent="${namespace}/base_link"
-  mass_rotor="${mass_rotor}"
-  radius_rotor="${radius_rotor}"
-  time_constant_up="${time_constant_up}"
-  time_constant_down="${time_constant_down}"
-  max_rot_velocity="${max_rot_velocity}"
-  motor_number="5"
-  rotor_drag_coefficient="${rotor_drag_coefficient}"
-  rolling_moment_coefficient="${rolling_moment_coefficient}"
-  color="Red"
-  use_own_mesh="false"
-  mesh="">
-  <origin xyz="-0.01948557158 0.01125 -0.03" rpy="0 0 0" />
-  <xacro:insert_block name="rotor_inertia" />
-</xacro:ARM3_macro>
+    <origin xyz="0.01948557158 0.01125 -0.03" rpy="0 0 0" />
+    <xacro:insert_block name="rotor_inertia" />
+  </xacro:ARM2_macro>
+  <!-- for ARM3 -->
+  <xacro:ARM3_macro
+    robot_namespace="${namespace}"
+    suffix="front_right"
+    direction="cw"
+    motor_constant="${motor_constant}"
+    moment_constant="${moment_constant}"
+    parent="${namespace}/base_link"
+    mass_rotor="${mass_rotor}"
+    radius_rotor="${radius_rotor}"
+    time_constant_up="${time_constant_up}"
+    time_constant_down="${time_constant_down}"
+    max_rot_velocity="${max_rot_velocity}"
+    motor_number="5"
+    rotor_drag_coefficient="${rotor_drag_coefficient}"
+    rolling_moment_coefficient="${rolling_moment_coefficient}"
+    color="Red"
+    use_own_mesh="false"
+    mesh="">
+    <origin xyz="-0.01948557158 0.01125 -0.03" rpy="0 0 0" />
+    <xacro:insert_block name="rotor_inertia" />
+  </xacro:ARM3_macro>
 </robot>
