Commit message: attached arm, included mesh files. Just have to allign angle/axis properly

File: urdf/firefly.xacro (robot description, xacro)
@@ -21,5 +21,5 @@
   <xacro:property name="rotor_velocity_slowdown_sim" value="10" />
   <xacro:property name="use_mesh_file" value="true" />
-  <xacro:property name="mesh_file" value="package://rotors_description/meshes/firefly.stl" />
+  <xacro:property name="mesh_file" value="package://swarm_collection/meshes/firefly.stl" />
   <xacro:property name="mass" value="1.5" /> <!-- [kg] -->
   <xacro:property name="body_width" value="0.1" /> <!-- [m] -->
@@ -185,4 +185,5 @@
     <xacro:insert_block name="rotor_inertia" />
   </xacro:vertical_rotor>
+<!-- for hub -->
   <xacro:hub_macro
     robot_namespace="${namespace}"
@@ -206,3 +207,69 @@
     <xacro:insert_block name="rotor_inertia" />
   </xacro:hub_macro>
+<!-- for ARM1 -->
+<xacro:ARM1_macro
+  robot_namespace="${namespace}"
+  suffix="front_right"
+  direction="cw"
+  motor_constant="${motor_constant}"
+  moment_constant="${moment_constant}"
+  parent="${namespace}/base_link"
+  mass_rotor="${mass_rotor}"
+  radius_rotor="${radius_rotor}"
+  time_constant_up="${time_constant_up}"
+  time_constant_down="${time_constant_down}"
+  max_rot_velocity="${max_rot_velocity}"
+  motor_number="5"
+  rotor_drag_coefficient="${rotor_drag_coefficient}"
+  rolling_moment_coefficient="${rolling_moment_coefficient}"
+  color="Red"
+  use_own_mesh="false"
+  mesh="">
+  <origin xyz="0 -0.0225 -0.03" rpy="0 0 0" />
+  <xacro:insert_block name="rotor_inertia" />
+</xacro:ARM1_macro>
+<!-- for ARM2 -->
+<xacro:ARM2_macro
+  robot_namespace="${namespace}"
+  suffix="front_right"
+  direction="cw"
+  motor_constant="${motor_constant}"
+  moment_constant="${moment_constant}"
+  parent="${namespace}/base_link"
+  mass_rotor="${mass_rotor}"
+  radius_rotor="${radius_rotor}"
+  time_constant_up="${time_constant_up}"
+  time_constant_down="${time_constant_down}"
+  max_rot_velocity="${max_rot_velocity}"
+  motor_number="5"
+  rotor_drag_coefficient="${rotor_drag_coefficient}"
+  rolling_moment_coefficient="${rolling_moment_coefficient}"
+  color="Red"
+  use_own_mesh="false"
+  mesh="">
+  <origin xyz="0.01948557158 0.01125 -0.03" rpy="0 0 0" />
+  <xacro:insert_block name="rotor_inertia" />
+</xacro:ARM2_macro>
+<!-- for ARM3 -->
+<xacro:ARM3_macro
+  robot_namespace="${namespace}"
+  suffix="front_right"
+  direction="cw"
+  motor_constant="${motor_constant}"
+  moment_constant="${moment_constant}"
+  parent="${namespace}/base_link"
+  mass_rotor="${mass_rotor}"
+  radius_rotor="${radius_rotor}"
+  time_constant_up="${time_constant_up}"
+  time_constant_down="${time_constant_down}"
+  max_rot_velocity="${max_rot_velocity}"
+  motor_number="5"
+  rotor_drag_coefficient="${rotor_drag_coefficient}"
+  rolling_moment_coefficient="${rolling_moment_coefficient}"
+  color="Red"
+  use_own_mesh="false"
+  mesh="">
+  <origin xyz="-0.01948557158 0.01125 -0.03" rpy="0 0 0" />
+  <xacro:insert_block name="rotor_inertia" />
+</xacro:ARM3_macro>
 </robot>

File: urdf/gripper.xacro (robot description, xacro)
@@ -1,4 +1,5 @@
 <?xml version="1.0"?>
 <robot xmlns:xacro="http://ros.org/wiki/xacro">
+<!--for hub -->
   <xacro:macro name="hub_macro"
     params="robot_namespace suffix direction motor_constant moment_constant parent mass_rotor radius_rotor time_constant_up time_constant_down max_rot_velocity motor_number rotor_drag_coefficient rolling_moment_coefficient color use_own_mesh mesh *origin *inertia">
@@ -34,3 +35,105 @@
     </link>
   </xacro:macro>
+  <!-- for ARM1 -->
+  <xacro:macro name="ARM1_macro"
+    params="robot_namespace suffix direction motor_constant moment_constant parent mass_rotor radius_rotor time_constant_up time_constant_down max_rot_velocity motor_number rotor_drag_coefficient rolling_moment_coefficient color use_own_mesh mesh *origin *inertia">
+    <joint name="${robot_namespace}/ARM1_joint" type="fixed">
+      <xacro:insert_block name="origin" />
+      <axis xyz="1 0 0" rpy="0 0 0" />
+      <parent link="${robot_namespace}/hub" />
+      <child link="${robot_namespace}/ARM1" />
+    </joint>
+    <link name="${robot_namespace}/ARM1">
+      <inertial>
+        <mass value="0.12781" /> <!-- [kg] -->
+        <inertia
+          ixx="0.00027224"
+          ixy="-6.26E-11"
+          ixz="-5.2198E-10"
+          iyy="0.00022223"
+          iyz="-7.6551E-05"
+          izz="6.3032E-05" />
+      </inertial>
+      <visual>
+        <origin  xyz="0 0 0" rpy="0 0 0" />
+        <geometry>
+            <mesh filename="package://swarm_collection/meshes/arm_link.STL" scale="1 1 1" />
+        </geometry>
+      </visual>
+      <collision>
+        <geometry>
+          <mesh
+            filename="package://swarm_collection/meshes/arm_link.STL" />
+        </geometry>
+      </collision>
+    </link>
+  </xacro:macro>
+  <!-- for ARM2 -->
+  <xacro:macro name="ARM2_macro"
+    params="robot_namespace suffix direction motor_constant moment_constant parent mass_rotor radius_rotor time_constant_up time_constant_down max_rot_velocity motor_number rotor_drag_coefficient rolling_moment_coefficient color use_own_mesh mesh *origin *inertia">
+    <joint name="${robot_namespace}/ARM2_joint" type="fixed">
+      <xacro:insert_block name="origin" />
+      <axis xyz="-0.5 0.86602540378 0" rpy="0 0 0" />
+      <parent link="${robot_namespace}/hub" />
+      <child link="${robot_namespace}/ARM2" />
+    </joint>
+    <link name="${robot_namespace}/ARM2">
+      <inertial>
+        <mass value="0.12781" /> <!-- [kg] -->
+        <inertia
+          ixx="0.00027224"
+          ixy="-6.26E-11"
+          ixz="-5.2198E-10"
+          iyy="0.00022223"
+          iyz="-7.6551E-05"
+          izz="6.3032E-05" />
+      </inertial>
+      <visual>
+        <origin  xyz="0 0 0" rpy="0 0 0" />
+        <geometry>
+            <mesh filename="package://swarm_collection/meshes/arm_link.STL" scale="1 1 1" />
+        </geometry>
+      </visual>
+      <collision>
+        <geometry>
+          <mesh
+            filename="package://swarm_collection/meshes/arm_link.STL" />
+        </geometry>
+      </collision>
+    </link>
+  </xacro:macro>
+  <!-- for ARM3 -->
+  <xacro:macro name="ARM3_macro"
+    params="robot_namespace suffix direction motor_constant moment_constant parent mass_rotor radius_rotor time_constant_up time_constant_down max_rot_velocity motor_number rotor_drag_coefficient rolling_moment_coefficient color use_own_mesh mesh *origin *inertia">
+    <joint name="${robot_namespace}/ARM3_joint" type="fixed">
+      <xacro:insert_block name="origin" />
+      <axis xyz="-0.5 -0.86602540378 0" rpy="0 0 0" />
+      <parent link="${robot_namespace}/hub" />
+      <child link="${robot_namespace}/ARM3" />
+    </joint>
+    <link name="${robot_namespace}/ARM3">
+      <inertial>
+        <mass value="0.12781" /> <!-- [kg] -->
+        <inertia
+          ixx="0.00027224"
+          ixy="-6.26E-11"
+          ixz="-5.2198E-10"
+          iyy="0.00022223"
+          iyz="-7.6551E-05"
+          izz="6.3032E-05" />
+      </inertial>
+      <visual>
+        <origin  xyz="0 0 0" rpy="0 0 0" />
+        <geometry>
+            <mesh filename="package://swarm_collection/meshes/arm_link.STL" scale="1 1 1" />
+        </geometry>
+      </visual>
+      <collision>
+        <geometry>
+          <mesh
+            filename="package://swarm_collection/meshes/arm_link.STL" />
+        </geometry>
+      </collision>
+    </link>
+  </xacro:macro>
 </robot>

Commit message: Added ROS Control for Gripper on Firefly

File: urdf/firefly.xacro (robot description, xacro)
@@ -210,69 +210,45 @@
   <!-- Pi/2 = 1.5708 -->
   <!-- Pi/6 = 0.5236 -->
-<!-- for ARM1 -->
-<xacro:ARM1_macro
+<!-- for arm1 -->
+<!-- <axis xyz="1 0 0" rpy="0 0 0" />
+<origin  xyz="0 0 0" rpy="0.7854 0 3.1416" /> -->
+<xacro:arm_macro
   robot_namespace="${namespace}"
-  suffix="front_right"
-  direction="cw"
-  motor_constant="${motor_constant}"
-  moment_constant="${moment_constant}"
   parent="${namespace}/base_link"
-  mass_rotor="${mass_rotor}"
-  radius_rotor="${radius_rotor}"
-  time_constant_up="${time_constant_up}"
-  time_constant_down="${time_constant_down}"
-  max_rot_velocity="${max_rot_velocity}"
-  motor_number="5"
-  rotor_drag_coefficient="${rotor_drag_coefficient}"
-  rolling_moment_coefficient="${rolling_moment_coefficient}"
-  color="Red"
-  use_own_mesh="false"
-  mesh="">
+  arm_number = "1"
+  axisxyz ="1 0 0"
+  axisrpy ="0 0 0"
+  originxyz = "0 0 0"
+  originrpy ="0.7854 0 3.1416"  >
   <origin xyz="0 -0.0225 -0.03" rpy="0 0 0" />
   <xacro:insert_block name="rotor_inertia" />
-</xacro:ARM1_macro>
-<!-- for ARM2 -->
-<xacro:ARM2_macro
+</xacro:arm_macro>
+<!-- for arm2 -->
+<!-- <axis xyz="-0.5 0.86602540378 0" rpy="0 0 0" />
+<origin  xyz="0 0 0" rpy="0.7854 0 -1.0472" /> -->
+<xacro:arm_macro
   robot_namespace="${namespace}"
-  suffix="front_right"
-  direction="cw"
-  motor_constant="${motor_constant}"
-  moment_constant="${moment_constant}"
   parent="${namespace}/base_link"
-  mass_rotor="${mass_rotor}"
-  radius_rotor="${radius_rotor}"
-  time_constant_up="${time_constant_up}"
-  time_constant_down="${time_constant_down}"
-  max_rot_velocity="${max_rot_velocity}"
-  motor_number="5"
-  rotor_drag_coefficient="${rotor_drag_coefficient}"
-  rolling_moment_coefficient="${rolling_moment_coefficient}"
-  color="Red"
-  use_own_mesh="false"
-  mesh="">
+  arm_number = "2"
+  axisxyz ="-0.5 0.86602540378 0"
+  axisrpy ="0 0 0"
+  originxyz = "0 0 0"
+  originrpy ="0.7854 0 -1.0472" >
   <origin xyz="0.01948557158 0.01125 -0.03" rpy="0 0 0" />
   <xacro:insert_block name="rotor_inertia" />
-</xacro:ARM2_macro>
-<!-- for ARM3 -->
-<xacro:ARM3_macro
+</xacro:arm_macro>
+<!-- for arm3 -->
+<!-- <axis xyz="-0.5 -0.86602540378 0" rpy="0 0 0" />
+<origin  xyz="0 0 0" rpy="0.7854 0 1.0472" /> -->
+<xacro:arm_macro
   robot_namespace="${namespace}"
-  suffix="front_right"
-  direction="cw"
-  motor_constant="${motor_constant}"
-  moment_constant="${moment_constant}"
   parent="${namespace}/base_link"
-  mass_rotor="${mass_rotor}"
-  radius_rotor="${radius_rotor}"
-  time_constant_up="${time_constant_up}"
-  time_constant_down="${time_constant_down}"
-  max_rot_velocity="${max_rot_velocity}"
-  motor_number="5"
-  rotor_drag_coefficient="${rotor_drag_coefficient}"
-  rolling_moment_coefficient="${rolling_moment_coefficient}"
-  color="Red"
-  use_own_mesh="false"
-  mesh="">
+  arm_number = "3"
+  axisxyz ="-0.5 -0.86602540378 0"
+  axisrpy ="0 0 0"
+  originxyz = "0 0 0"
+  originrpy ="0.7854 0 1.0472" >
   <origin xyz="-0.01948557158 0.01125 -0.03" rpy="0 0 0" />
   <xacro:insert_block name="rotor_inertia" />
-</xacro:ARM3_macro>
+</xacro:arm_macro>
 </robot>

File: urdf/gripper.xacro (robot description, xacro)
@@ -10,5 +10,5 @@
   iyz="3.7001E-10"
   izz="4.5243E-05" /> -->
-  <!-- Inertia of Arm
+  <!-- Inertia of arm
  <inertia
     ixx="0.00027224"
@@ -52,15 +52,23 @@
       </collision>
     </link>
+    <gazebo>
+        <plugin name="${robot_namespace}_gripper_ros_control" filename="libgazebo_ros_control.so">
+    	  <!--this is the namespace in the yaml file-->
+          <robotNamespace>/firefly</robotNamespace>
+          <!--The two lines below came from: https://answers.ros.org/question/292444/gazebo_ros_control-plugin-gazeboroscontrolplugin-missing-legacymodens-defaultrobothwsim/-->
+          <robotSimType>gazebo_ros_control/DefaultRobotHWSim</robotSimType>
+        </plugin>
+    </gazebo>
   </xacro:macro>
-  <!-- for ARM1 -->
-  <xacro:macro name="ARM1_macro"
-    params="robot_namespace suffix direction motor_constant moment_constant parent mass_rotor radius_rotor time_constant_up time_constant_down max_rot_velocity motor_number rotor_drag_coefficient rolling_moment_coefficient color use_own_mesh mesh *origin *inertia">
-    <joint name="${robot_namespace}/ARM1_joint" type="fixed">
+  <!-- for arm1 -->
+  <xacro:macro name="arm_macro"
+    params="robot_namespace parent arm_number axisxyz axisrpy originxyz originrpy *origin *inertia">
+    <joint name="${robot_namespace}/arm${arm_number}_joint" type="continuous">
       <xacro:insert_block name="origin" />
-      <axis xyz="1 0 0" rpy="0 0 0" />
+      <axis xyz= "${axisxyz}" rpy="${axisrpy}" />
       <parent link="${robot_namespace}/hub" />
-      <child link="${robot_namespace}/ARM1" />
+      <child link="${robot_namespace}/arm${arm_number}" />
     </joint>
-    <link name="${robot_namespace}/ARM1">
+    <link name="${robot_namespace}/arm${arm_number}">
       <inertial>
         <mass value="0.05" /> <!-- [kg] -->
@@ -74,5 +82,5 @@
       </inertial>
       <visual>
-        <origin  xyz="0 0 0" rpy="0.7854 0 3.1416" />
+        <origin  xyz= "${originxyz}" rpy="${originrpy}"  />
         <geometry>
             <mesh filename="package://swarm_collection/meshes/arm_link.STL" scale="1 1 1" />
@@ -80,5 +88,5 @@
       </visual>
       <collision>
-        <origin  xyz="0 0 0" rpy="0.7854 0 3.1416" />
+        <origin  xyz= "${originxyz}" rpy="${originrpy}"  />
         <geometry>
           <mesh
@@ -87,74 +95,18 @@
       </collision>
     </link>
-  </xacro:macro>
-  <!-- for ARM2 -->
-  <xacro:macro name="ARM2_macro"
-    params="robot_namespace suffix direction motor_constant moment_constant parent mass_rotor radius_rotor time_constant_up time_constant_down max_rot_velocity motor_number rotor_drag_coefficient rolling_moment_coefficient color use_own_mesh mesh *origin *inertia">
-    <joint name="${robot_namespace}/ARM2_joint" type="fixed">
-      <xacro:insert_block name="origin" />
-      <axis xyz="-0.5 0.86602540378 0" rpy="0 0 0" />
-      <parent link="${robot_namespace}/hub" />
-      <child link="${robot_namespace}/ARM2" />
-    </joint>
-    <link name="${robot_namespace}/ARM2">
-      <inertial>
-        <mass value="0.05" /> <!-- [kg] -->
-        <inertia
-          ixx="2714.030518E-6"
-          ixy="0.000007E-6"
-          ixz="0.000038E-6"
-          iyy="2216.979248E-6"
-          iyz="-762.669067E-6"
-          izz="627.139465E-6" />
-      </inertial>
-      <visual>
-        <origin  xyz="0 0 0" rpy="0.7854 0 -1.0472" />
-        <geometry>
-            <mesh filename="package://swarm_collection/meshes/arm_link.STL" scale="1 1 1" />
-        </geometry>
-      </visual>
-      <collision>
-        <origin  xyz="0 0 0" rpy="0.7854 0 -1.0472" />
-        <geometry>
-          <mesh
-            filename="package://swarm_collection/meshes/arm_link.STL" />
-        </geometry>
-      </collision>
-    </link>
-  </xacro:macro>
-  <!-- for ARM3 -->
-  <xacro:macro name="ARM3_macro"
-    params="robot_namespace suffix direction motor_constant moment_constant parent mass_rotor radius_rotor time_constant_up time_constant_down max_rot_velocity motor_number rotor_drag_coefficient rolling_moment_coefficient color use_own_mesh mesh *origin *inertia">
-    <joint name="${robot_namespace}/ARM3_joint" type="fixed">
-      <xacro:insert_block name="origin" />
-      <axis xyz="-0.5 -0.86602540378 0" rpy="0 0 0" />
-      <parent link="${robot_namespace}/hub" />
-      <child link="${robot_namespace}/ARM3" />
-    </joint>
-    <link name="${robot_namespace}/ARM3">
-      <inertial>
-        <mass value="0.05" /> <!-- [kg] -->
-        <inertia
-          ixx="2714.030518E-6"
-          ixy="0.000007E-6"
-          ixz="0.000038E-6"
-          iyy="2216.979248E-6"
-          iyz="-762.669067E-6"
-          izz="627.139465E-6" />
-      </inertial>
-      <visual>
-        <origin  xyz="0 0 0" rpy="0.7854 0 1.0472" />
-        <geometry>
-            <mesh filename="package://swarm_collection/meshes/arm_link.STL" scale="1 1 1" />
-        </geometry>
-      </visual>
-      <collision>
-        <origin  xyz="0 0 0" rpy="0.7854 0 1.0472" />
-        <geometry>
-          <mesh
-            filename="package://swarm_collection/meshes/arm_link.STL" />
-        </geometry>
-      </collision>
-    </link>
+    <!-- transmission is the ability to define the ros controller used to control the joint. -->
+    <transmission name="${robot_namespace}/arm${arm_number}_joint_trans">
+      <type>transmission_interface/SimpleTransmission</type>
+      <actuator name="motor${arm_number}">
+        <!--<hardwareInterface>hardware_interface/EffortJointInterface</hardwareInterface> -->
+        <mechanicalReduction>1</mechanicalReduction>
+      </actuator>
+      <joint name="${robot_namespace}/arm${arm_number}_joint">
+        <!--lets use a postion type interface, which is a mechanism for ros_control
+            to communicate with hardware. See: https://wiki.ros.org/ros_control-->
+        <!--hardwareInterface>hardware_interface/PositionJointInterface</hardwareInterface-->
+        <hardwareInterface>hardware_interface/PositionJointInterface</hardwareInterface>
+      </joint>
+    </transmission>
   </xacro:macro>
 </robot>
